Commit message: Gazebo sim up and running

File: install/robomop_description/share/robomop_description/urdf/common/inertials.xacro (robot description, xacro)
@@ -1 +1 @@
-/home/robomop/robomop_ws/src/robomop_description/urdf/common/inertials.xacro
+/home/robmop-dev/robomop_ws/robomop/src/robomop_description/urdf/common/inertials.xacro

File: install/robomop_description/share/robomop_description/urdf/common/materials.xacro (robot description, xacro)
@@ -1 +1 @@
-/home/robomop/robomop_ws/src/robomop_description/urdf/common/materials.xacro
+/home/robmop-dev/robomop_ws/robomop/src/robomop_description/urdf/common/materials.xacro

File: install/robomop_description/share/robomop_description/urdf/robomop.urdf.xacro (robot description, xacro)
@@ -1 +1 @@
-/home/robomop/robomop_ws/src/robomop_description/urdf/robomop.urdf.xacro
+/home/robmop-dev/robomop_ws/robomop/src/robomop_description/urdf/robomop.urdf.xacro

File: install/robomop_description/share/robomop_description/urdf/robomop/robomop_macro.xacro (robot description, xacro)
@@ -1 +1 @@
-/home/robomop/robomop_ws/src/robomop_description/urdf/robomop/robomop_macro.xacro
+/home/robmop-dev/robomop_ws/robomop/src/robomop_description/urdf/robomop/robomop_macro.xacro

File: src/robomop_description/urdf/robomop.urdf.xacro (robot description, xacro)
@@ -1,14 +1,33 @@
-<robot xmlns:xacro="http://www.ros.org/wiki/xacro" name="robomop">
-    <!-- Robot Parameters -->
+<?xml version="1.0"?>
+<robot xmlns:xacro="http://ros.org/wiki/xacro" name="robomop">
+    <!-- ============================
+         Robot Parameters
+    ============================= -->
+    <!-- Mass Properties -->
+    <xacro:property name="chassis_mass" value="1.0" />   <!-- 1 kg -->
+    <xacro:property name="wheel_mass" value="0.1" />      <!-- 0.1 kg each -->
+    <xacro:property name="brush_mass" value="0.05" />     <!-- 0.05 kg each -->
+    <!-- Geometric Parameters -->
+    <xacro:property name="chassis_length" value="0.35306" />
+    <xacro:property name="chassis_width" value="0.4064" />
+    <xacro:property name="chassis_height" value="0.144" />
+    <xacro:property name="wheel_radius" value="0.08" />
+    <xacro:property name="wheel_length" value="0.022" />
+    <xacro:property name="brush_radius" value="0.08" />
+    <xacro:property name="brush_length" value="0.01" />
+    <!-- Wheel Offsets -->
     <xacro:property name="wheel_x_offset" value="-0.062" />
     <xacro:property name="wheel_y_offset" value="0.175" />
     <xacro:property name="wheel_z_offset" value="0.043" />
-    <xacro:property name="wheel_mass" value="3.62874" />
-    <xacro:property name="chassis_mass" value="1.36078" />
-    <!-- Xacro Common Files -->
+    <!-- Common Files -->
     <xacro:include filename="$(find robomop_description)/urdf/common/inertials.xacro" />
     <xacro:include filename="$(find robomop_description)/urdf/common/materials.xacro" />
-    <!-- Robot Links -->
-    <link name="base_link" />
+    <!-- ============================
+         Define Links
+    ============================= -->
+    <!-- Base Link -->
+    <link name="base_link">
+    </link>
+    <!-- Chassis Link -->
     <link name="chassis_link">
         <visual>
@@ -25,85 +44,58 @@
             </geometry>
         </collision>
-        <inertial>
-            <origin xyz="0.0 0.0 0.02" rpy="0 0 0"/>
-            <mass value="${chassis_mass}" />
-            <inertia ixx="0.006453" ixy="0"  ixz="0" iyy="0.0117" iyz="0" izz="0.015812" />
-        </inertial>
+        <!-- Using Box Inertial Macro -->
+        <xacro:box_inertial x="${chassis_length}" y="${chassis_width}" z="${chassis_height}" mass="${chassis_mass}">
+            <origin xyz="0.008 0.0 0.072" rpy="0 0 0"/>
+        </xacro:box_inertial>
     </link>
-    <link name="rl_wheel_link">
-        <visual>
-            <origin xyz="0 0 0"/>
-            <geometry>
-                <mesh filename="file://$(find robomop_description)/meshes/visual/robomop_wheel.stl" scale="0.001 0.001 0.001"/>
-            </geometry>
-            <material name="white" />
-        </visual>
-        <collision>
-            <origin xyz="0 0 0"/>
-            <geometry>
-                <mesh filename="file://$(find robomop_description)/meshes/visual/robomop_wheel.stl" scale="0.001 0.001 0.001"/>
-            </geometry>
-        </collision>
-        <inertial>
-            <origin xyz="0 0 0" rpy="0 0 0" />
-            <mass value="${wheel_mass}" />
-            <inertia ixx="0.008093" ixy="0"  ixz="0" iyy="0.014226" iyz="0" izz="0.008093" />
-        </inertial>
-        <mu>5.0</mu>
-    </link>
-    <link name="rr_wheel_link">
-        <visual>
-            <origin xyz="0 0 0"/>
-            <geometry>
-                <mesh filename="file://$(find robomop_description)/meshes/visual/robomop_wheel.stl" scale="0.001 0.001 0.001"/>
-            </geometry>
-            <material name="white" />
-        </visual>
-        <collision>
-            <origin xyz="0 0 0"/>
-            <geometry>
-                <mesh filename="file://$(find robomop_description)/meshes/visual/robomop_wheel.stl" scale="0.001 0.001 0.001"/>
-            </geometry>
-        </collision>
-        <inertial>
-            <origin xyz="0 0 0" rpy="0 0 0" />
-            <mass value="${wheel_mass}" />
-            <inertia ixx="0.008093" ixy="0"  ixz="0" iyy="0.014226" iyz="0" izz="0.008093" />
-        </inertial>
-        <mu>5.0</mu>
-    </link>
-    <link name="right_brush">
-        <visual>
-            <origin xyz="0 0 0"/>
-            <geometry>
-                <mesh filename="file://$(find robomop_description)/meshes/visual/robomop_brush.stl" scale="0.001 0.001 0.001"/>
-            </geometry>
-            <material name="dark_grey" />
-        </visual>
-        <collision>
-            <origin xyz="0 0 0"/>
-            <geometry>
-                <mesh filename="file://$(find robomop_description)/meshes/visual/robomop_brush.stl" scale="0.001 0.001 0.001"/>
-            </geometry>
-        </collision>
-    </link>
-    <link name="left_brush">
-        <visual>
-            <origin xyz="0 0 0"/>
-            <geometry>
-                <mesh filename="file://$(find robomop_description)/meshes/visual/robomop_brush.stl" scale="0.001 0.001 0.001"/>
-            </geometry>
-            <material name="dark_grey" />
-        </visual>
-        <collision>
-            <origin xyz="0 0 0"/>
-            <geometry>
-                <mesh filename="file://$(find robomop_description)/meshes/visual/robomop_brush.stl" scale="0.001 0.001 0.001"/>
-            </geometry>
-        </collision>
-    </link>
+    <!-- Wheel Links Macro -->
+    <xacro:macro name="wheel_link" params="name material">
+        <link name="${name}">
+            <visual>
+                <origin xyz="0 0 0"/>
+                <geometry>
+                    <mesh filename="file://$(find robomop_description)/meshes/visual/robomop_wheel.stl" scale="0.001 0.001 0.001"/>
+                </geometry>
+                <material name="${material}" />
+            </visual>
+            <collision>
+                <origin xyz="0 0 0"/>
+                <geometry>
+                    <mesh filename="file://$(find robomop_description)/meshes/visual/robomop_wheel.stl" scale="0.001 0.001 0.001"/>
+                </geometry>
+            </collision>
+            <!-- Using Cylinder Inertial Macro -->
+            <xacro:cylinder_inertial radius="${wheel_radius}" length="${wheel_length}" mass="${wheel_mass}">
+                <origin xyz="0.0 0.0111 0" rpy="1.57 0 0"/>
+            </xacro:cylinder_inertial>
+            <mu>5.0</mu>
+        </link>
+    </xacro:macro>
+    <!-- Define RL and RR Wheels -->
+    <xacro:wheel_link name="rl_wheel_link" material="white" />
+    <xacro:wheel_link name="rr_wheel_link" material="white" />
+    <!-- Brush Links Macro -->
+    <xacro:macro name="brush_link" params="name material">
+        <link name="${name}">
+            <visual>
+                <origin xyz="0 0 0"/>
+                <geometry>
+                    <mesh filename="file://$(find robomop_description)/meshes/visual/robomop_brush.stl" scale="0.001 0.001 0.001"/>
+                </geometry>
+                <material name="${material}" />
+            </visual>
+            <!-- Using Sphere Inertial Macro -->
+            <xacro:cylinder_inertial radius="${brush_radius}" length="${brush_length}" mass="${brush_mass}">
+                <origin xyz="0 0 0" rpy="0 0 0"/>
+            </xacro:cylinder_inertial>
+        </link>
+    </xacro:macro>
+    <!-- Define Left and Right Brushes -->
+    <xacro:brush_link name="left_brush" material="dark_grey" />
+    <xacro:brush_link name="right_brush" material="dark_grey" />
+    <!-- Caster Housing Link (No Inertial) -->
     <link name="caster_housing">
         <visual>
-            <origin xyz="0 ${0.047/2} 0" rpy="0 3.14 1.57"/>
+            <origin xyz="0 0.0235 0" rpy="0 3.14 1.57"/> <!-- 0.047/2 = 0.0235 -->
             <geometry>
                 <mesh filename="file://$(find robomop_description)/meshes/visual/robomop_caster.stl" scale="0.001 0.001 0.001"/>
@@ -112,5 +104,5 @@
         </visual>
         <collision>
-            <origin xyz="0 ${0.047/2} 0" rpy="0 3.14 1.57"/>
+            <origin xyz="0 0.0235 0" rpy="0 3.14 1.57"/>
             <geometry>
                 <mesh filename="file://$(find robomop_description)/meshes/visual/robomop_caster.stl" scale="0.001 0.001 0.001"/>
@@ -118,7 +110,8 @@
         </collision>
     </link>
+    <!-- Caster Wheel Link (No Inertial) -->
     <link name="caster_wheel">
         <visual>
-            <origin xyz="${(-23.619)/1000} ${16.211/1000} ${(-13.5)/1000}"/>
+            <origin xyz="-0.023619 0.016211 -0.0135"/> <!-- Converted to meters -->
             <geometry>
                 <mesh filename="file://$(find robomop_description)/meshes/visual/robomop_caster_wheel.stl" scale="0.001 0.001 0.001"/>
@@ -135,10 +128,14 @@
     <!-- Lidar Link -->
     <xacro:include filename="$(find ldlidar_node)/urdf/ldlidar_descr.urdf.xml" />
-    <!-- Joints -->
+    <!-- ============================
+         Define Joints
+    ============================= -->
+    <!-- Fixed Joint: Base to Chassis -->
     <joint name="base_to_chassis" type="fixed">
         <parent link="base_link"/>
         <child link="chassis_link"/>
-        <origin xyz="0 0 ${0.006 + 0.018}"/>
-    </joint>
+        <origin xyz="0 0 0.024" rpy="0 0 0"/> <!-- 0.006 + 0.018 -->
+    </joint>
+    <!-- Continuous Joints: Wheels to Chassis -->
     <joint name="rl_wheel_to_chassis" type="continuous">
         <parent link="chassis_link"/>
@@ -153,4 +150,5 @@
         <origin xyz="${wheel_x_offset} ${-wheel_y_offset - 0.022} ${wheel_z_offset}" rpy="0 0 0" />
     </joint>
+    <!-- Continuous Joints: Brushes to Chassis -->
     <joint name="right_brush_to_chassis" type="continuous">
         <parent link="chassis_link"/>
@@ -165,14 +163,16 @@
         <origin xyz="0.1067 0.0762 -0.016" rpy="0 0 0" />
     </joint>
+    <!-- Fixed Joints: Caster Housing and Wheel -->
     <joint name="caster_housing_to_chassis" type="fixed">
         <parent link="chassis_link"/>
         <child link="caster_housing"/>
-        <origin xyz="${(149.9 - 23.62)/1000} ${0} ${(-14.00)/1000}" rpy="0 0 0" />
+        <origin xyz="0.12628 0  -0.014" rpy="0 0 0"/> <!-- (149.9 - 23.62)/1000 = 0.12628 -->
     </joint>
     <joint name="caster_wheel_to_housing" type="fixed">
         <parent link="caster_housing"/>
         <child link="caster_wheel"/>
-        <origin xyz="${16.211/1000} 0 ${(-13)/1000}" rpy="0 0 0" />
-    </joint>
+        <origin xyz="0.016211 0 -0.013" rpy="0 0 0"/> <!-- 16.211/1000, 0, -13/1000 -->
+    </joint>
+    <!-- Fixed Joint: Lidar to Chassis -->
     <joint name="lidar_to_chassis" type="fixed">
         <parent link="chassis_link"/>
@@ -180,5 +180,34 @@
         <origin xyz="0.019 0 0.138" rpy="0 0 0" />
     </joint>
+    <!-- ============================
+        ros2_control Transmissions
+    ============================= -->
+    <!-- Transmission for RL Wheel -->
+    <transmission name="rl_wheel_trans">
+        <type>transmission_interface/SimpleTransmission</type>
+        <joint name="rl_wheel_to_chassis">
+            <hardware_interface>hardware_interface/VelocityJointInterface</hardware_interface>
+        </joint>
+        <actuator name="rl_wheel_motor">
+            <hardware_interface>hardware_interface/VelocityJointInterface</hardware_interface>
+            <mechanical_reduction>1</mechanical_reduction>
+        </actuator>
+    </transmission>
+    <!-- Transmission for RR Wheel -->
+    <transmission name="rr_wheel_trans">
+        <type>transmission_interface/SimpleTransmission</type>
+        <joint name="rr_wheel_to_chassis">
+            <hardware_interface>hardware_interface/VelocityJointInterface</hardware_interface>
+        </joint>
+        <actuator name="rr_wheel_motor">
+            <hardware_interface>hardware_interface/VelocityJointInterface</hardware_interface>
+            <mechanical_reduction>1</mechanical_reduction>
+        </actuator>
+    </transmission>
+    <!-- ============================
+         Gazebo Plugins
+    ============================= -->
     <gazebo>
+        <!-- DiffDrive Plugin -->
         <plugin name="ignition::gazebo::systems::DiffDrive" filename="ignition-gazebo-diff-drive-system">
             <num_wheel_pairs>2</num_wheel_pairs>
@@ -193,5 +222,5 @@
             <max_angular_acceleration>4</max_angular_acceleration>
             <min_angular_acceleration>-4</min_angular_acceleration>
-            <!-- Output -->
+            <!-- Output Frames -->
             <frame_id>odom</frame_id>
             <child_frame_id>base_link</child_frame_id>
@@ -201,11 +230,17 @@
             <tf_topic>/tf_gazebo</tf_topic>
         </plugin>
+        <!-- Joint State Publisher Plugin -->
         <plugin filename="ignition-gazebo-joint-state-publisher-system" name="ignition::gazebo::systems::JointStatePublisher">
             <topic>/joint_states</topic>
         </plugin>
+        <!-- Sensors Plugin -->
         <plugin filename="libignition-gazebo-sensors-system.so" name="ignition::gazebo::systems::Sensors">
             <render_engine>ogre2</render_engine>
         </plugin>
     </gazebo>
+    <!-- ============================
+         Gazebo Contact Parameters
+    ============================= -->
+    <!-- RL Wheel Contact -->
     <gazebo reference="rl_wheel_link">
         <mu1 value="200.0" />
@@ -215,4 +250,5 @@
         <minDepth>0.005</minDepth>
     </gazebo>
+    <!-- RR Wheel Contact -->
     <gazebo reference="rr_wheel_link">
         <mu1 value="200.0" />
@@ -222,4 +258,14 @@
         <minDepth>0.005</minDepth>
     </gazebo>
+    <!-- Caster Wheel Contact (Including Brushes) -->
+    <gazebo reference="caster_wheel">
+        <!-- Combine caster wheel and brushes friction -->
+        <mu1 value="50.0" /> <!-- Lower friction -->
+        <mu2 value="50.0" />
+        <kp  value="500000.0" /> <!-- Lower stiffness -->
+        <kd  value="0.5" />
+        <minDepth>0.005</minDepth>
+    </gazebo>
+    <!-- Lidar Sensor Configuration -->
     <gazebo reference="ldlidar_base">
         <sensor name='gpu_lidar' type='gpu_lidar'>
@@ -230,21 +276,21 @@
             <lidar>
                 <scan>
-                <horizontal>
-                    <samples>640</samples>
-                    <resolution>1</resolution>
-                    <min_angle>-3.14159</min_angle>
-                    <max_angle>3.14159</max_angle>
-                </horizontal>
-                <vertical>
-                    <samples>1</samples>
-                    <resolution>1</resolution>
-                    <min_angle>0.0</min_angle>
-                    <max_angle>0.0</max_angle>
-                </vertical>
+                    <horizontal>
+                        <samples>640</samples>
+                        <resolution>1</resolution>
+                        <min_angle>-3.14159</min_angle>
+                        <max_angle>3.14159</max_angle>
+                    </horizontal>
+                    <vertical>
+                        <samples>1</samples>
+                        <resolution>1</resolution>
+                        <min_angle>0.0</min_angle>
+                        <max_angle>0.0</max_angle>
+                    </vertical>
                 </scan>
                 <range>
-                <min>0.15</min>
-                <max>12.0</max>
-                <resolution>0.01</resolution>
+                    <min>0.15</min>
+                    <max>12.0</max>
+                    <resolution>0.01</resolution>
                 </range>
             </lidar>
