Commit message: Update URDF

File: src/robomop_description/urdf/robomop.urdf.xacro (robot description, xacro)
@@ -13,5 +13,5 @@
             <origin xyz="0.01 0.02 0" rpy="0 -0 1.5708" />
             <geometry>
-                <mesh filename="file://$(find robomop_description)/meshes/visual/robomop_assy.stl"/>
+                <mesh filename="file://$(find robomop_description)/meshes/visual/robomop_shell.stl" scale="0.001 0.001 0.001"/>
             </geometry>
         </visual>
@@ -19,5 +19,5 @@
             <origin xyz="0.01 0.02 0" rpy="0 -0 1.5708" />
             <geometry>
-                <mesh filename="file://$(find robomop_description)/meshes/visual/robomop_assy.stl"/>
+                <mesh filename="file://$(find robomop_description)/meshes/visual/robomop_shell.stl" scale="0.001 0.001 0.001"/>
             </geometry>
         </collision>
@@ -28,21 +28,16 @@
         </inertial>
     </link>
-    <joint name="base_to_chassis" type="fixed">
-        <parent link="base_link"/>
-        <child link="chassis_link"/>
-        <origin xyz="0 0 0.0965"/>
-    </joint>
     <link name="rl_wheel_link">
         <visual>
             <origin xyz="0 0 0" rpy="1.57 3.1415 0" />
-            <!-- <geometry>
-                <mesh filename="file://$(find roverrobotics_description)/meshes/hub_6.5in.dae"/>
-            </geometry> -->
+            <geometry>
+                <mesh filename="file://$(find robomop_description)/meshes/visual/robomop_wheel.stl" scale="0.001 0.001 0.001"/>
+            </geometry>
         </visual>
         <collision>
             <origin xyz="0 0 0" rpy="1.57 3.1415 0" />
-            <!-- <geometry>
-                <mesh filename="file://$(find roverrobotics_description)/meshes/hub_6.5in.dae"/>
-            </geometry> -->
+            <geometry>
+                <mesh filename="file://$(find robomop_description)/meshes/visual/robomop_wheel.stl" scale="0.001 0.001 0.001"/>
+            </geometry>
         </collision>
         <inertial>
@@ -53,22 +48,16 @@
         <mu>5.0</mu>
     </link>
-    <joint name="rl_wheel_to_chassis" type="continuous">
-        <parent link="base_link"/>
-        <child link="rl_wheel_link"/>
-        <axis xyz="0 1 0"/>
-        <origin xyz="${-wheel_x_offset} ${wheel_y_offset} ${wheel_z_offset}"/>
-    </joint>
     <link name="rr_wheel_link">
         <visual>
             <origin xyz="0 0 0" rpy="1.57 3.1415 3.1415" />
-            <!-- <geometry>
-                <mesh filename="file://$(find roverrobotics_description)/meshes/hub_6.5in.dae"/>
-            </geometry> -->
+            <geometry>
+                <mesh filename="file://$(find robomop_description)/meshes/visual/robomop_wheel.stl" scale="0.001 0.001 0.001"/>
+            </geometry>
         </visual>
         <collision>
             <origin xyz="0 0 0" rpy="1.57 3.1415 3.1415" />
-            <!-- <geometry>
-                <mesh filename="file://$(find roverrobotics_description)/meshes/hub_6.5in.dae"/>
-            </geometry> -->
+            <geometry>
+                <mesh filename="file://$(find robomop_description)/meshes/visual/robomop_wheel.stl" scale="0.001 0.001 0.001"/>
+            </geometry>
         </collision>
         <inertial>
@@ -79,9 +68,20 @@
         <mu>5.0</mu>
     </link>
+    <joint name="base_to_chassis" type="fixed">
+        <parent link="base_link"/>
+        <child link="chassis_link"/>
+        <origin xyz="0 0 0.1"/>
+    </joint>
+    <joint name="rl_wheel_to_chassis" type="continuous">
+        <parent link="chassis_link"/>
+        <child link="rl_wheel_link"/>
+        <axis xyz="0 1 0"/>
+        <origin xyz="0 0 0"/>
+    </joint>
     <joint name="rr_wheel_to_chassis" type="continuous">
-        <parent link="base_link"/>
+        <parent link="chassis_link"/>
         <child link="rr_wheel_link"/>
         <axis xyz="0 1 0"/>
-        <origin xyz="${-wheel_x_offset} ${-wheel_y_offset} ${wheel_z_offset}"/>
+        <origin xyz="0 0 0"/>
     </joint>
     <gazebo>

Commit message: Add robomop lidar and sim plugin

File: src/robomop_description/urdf/robomop.urdf.xacro (robot description, xacro)
@@ -1,21 +1,24 @@
 <robot xmlns:xacro="http://www.ros.org/wiki/xacro" name="robomop">
     <!-- Robot Parameters -->
-    <xacro:property name="wheel_z_offset" value="-0.0155" />
-    <xacro:property name="wheel_x_offset" value="0.11" />
-    <xacro:property name="front_wheel_x_offset" value="0.006" />
-    <xacro:property name="wheel_y_offset" value="0.155" />
+    <xacro:property name="wheel_x_offset" value="-0.062" />
+    <xacro:property name="wheel_y_offset" value="0.175" />
+    <xacro:property name="wheel_z_offset" value="0.043" />
     <xacro:property name="wheel_mass" value="3.62874" />
     <xacro:property name="chassis_mass" value="1.36078" />
-    <!-- Robot Description -->
+    <!-- Xacro Common Files -->
+    <xacro:include filename="$(find robomop_description)/urdf/common/inertials.xacro" />
+    <xacro:include filename="$(find robomop_description)/urdf/common/materials.xacro" />
+    <!-- Robot Links -->
     <link name="base_link" />
     <link name="chassis_link">
         <visual>
-            <origin xyz="0.01 0.02 0" rpy="0 -0 1.5708" />
+            <origin xyz="0 0 0" rpy="0 0 0" />
             <geometry>
                 <mesh filename="file://$(find robomop_description)/meshes/visual/robomop_shell.stl" scale="0.001 0.001 0.001"/>
             </geometry>
+            <material name="light_grey" />
         </visual>
         <collision>
-            <origin xyz="0.01 0.02 0" rpy="0 -0 1.5708" />
+            <origin xyz="0.0 0.0 0" rpy="0 0 0" />
             <geometry>
                 <mesh filename="file://$(find robomop_description)/meshes/visual/robomop_shell.stl" scale="0.001 0.001 0.001"/>
@@ -30,11 +33,12 @@
     <link name="rl_wheel_link">
         <visual>
-            <origin xyz="0 0 0" rpy="1.57 3.1415 0" />
+            <origin xyz="0 0 0"/>
             <geometry>
                 <mesh filename="file://$(find robomop_description)/meshes/visual/robomop_wheel.stl" scale="0.001 0.001 0.001"/>
             </geometry>
+            <material name="white" />
         </visual>
         <collision>
-            <origin xyz="0 0 0" rpy="1.57 3.1415 0" />
+            <origin xyz="0 0 0"/>
             <geometry>
                 <mesh filename="file://$(find robomop_description)/meshes/visual/robomop_wheel.stl" scale="0.001 0.001 0.001"/>
@@ -50,11 +54,12 @@
     <link name="rr_wheel_link">
         <visual>
-            <origin xyz="0 0 0" rpy="1.57 3.1415 3.1415" />
+            <origin xyz="0 0 0"/>
             <geometry>
                 <mesh filename="file://$(find robomop_description)/meshes/visual/robomop_wheel.stl" scale="0.001 0.001 0.001"/>
             </geometry>
+            <material name="white" />
         </visual>
         <collision>
-            <origin xyz="0 0 0" rpy="1.57 3.1415 3.1415" />
+            <origin xyz="0 0 0"/>
             <geometry>
                 <mesh filename="file://$(find robomop_description)/meshes/visual/robomop_wheel.stl" scale="0.001 0.001 0.001"/>
@@ -68,8 +73,11 @@
         <mu>5.0</mu>
     </link>
+    <!-- Lidar Link -->
+    <xacro:include filename="$(find ldlidar_node)/urdf/ldlidar_descr.urdf.xml" />
+    <!-- Joints -->
     <joint name="base_to_chassis" type="fixed">
         <parent link="base_link"/>
         <child link="chassis_link"/>
-        <origin xyz="0 0 0.1"/>
+        <origin xyz="0 0 ${0.006 + 0.018}"/>
     </joint>
     <joint name="rl_wheel_to_chassis" type="continuous">
@@ -77,5 +85,5 @@
         <child link="rl_wheel_link"/>
         <axis xyz="0 1 0"/>
-        <origin xyz="0 0 0"/>
+        <origin xyz="${wheel_x_offset} ${wheel_y_offset} ${wheel_z_offset}" rpy="0 0 0" />
     </joint>
     <joint name="rr_wheel_to_chassis" type="continuous">
@@ -83,5 +91,10 @@
         <child link="rr_wheel_link"/>
         <axis xyz="0 1 0"/>
-        <origin xyz="0 0 0"/>
+        <origin xyz="${wheel_x_offset} ${-wheel_y_offset - 0.022} ${wheel_z_offset}" rpy="0 0 0" />
+    </joint>
+    <joint name="lidar_to_chassis" type="fixed">
+        <parent link="chassis_link"/>
+        <child link="ldlidar_base"/>
+        <origin xyz="0.019 0 0.138" rpy="0 0 0" />
     </joint>
     <gazebo>
@@ -109,4 +122,7 @@
             <topic>/joint_states</topic>
         </plugin>
+        <plugin filename="libignition-gazebo-sensors-system.so" name="ignition::gazebo::systems::Sensors">
+            <render_engine>ogre2</render_engine>
+        </plugin>
     </gazebo>
     <gazebo reference="rl_wheel_link">
@@ -124,3 +140,33 @@
         <minDepth>0.005</minDepth>
     </gazebo>
+    <gazebo reference="ldlidar_base">
+        <sensor name='gpu_lidar' type='gpu_lidar'>
+            <pose>0 0 0 0 0 0</pose>
+            <topic>scan</topic>
+            <ignition_frame_id>ldlidar_base</ignition_frame_id>
+            <update_rate>10</update_rate>
+            <lidar>
+                <scan>
+                <horizontal>
+                    <samples>640</samples>
+                    <resolution>1</resolution>
+                    <min_angle>-3.14159</min_angle>
+                    <max_angle>3.14159</max_angle>
+                </horizontal>
+                <vertical>
+                    <samples>1</samples>
+                    <resolution>1</resolution>
+                    <min_angle>0.0</min_angle>
+                    <max_angle>0.0</max_angle>
+                </vertical>
+                </scan>
+                <range>
+                <min>0.15</min>
+                <max>12.0</max>
+                <resolution>0.01</resolution>
+                </range>
+            </lidar>
+            <visualize>true</visualize>
+        </sensor>
+    </gazebo>
 </robot>

Commit message: Finish URDF definition

File: src/robomop_description/urdf/robomop.urdf.xacro (robot description, xacro)
@@ -73,4 +73,64 @@
         <mu>5.0</mu>
     </link>
+    <link name="right_brush">
+        <visual>
+            <origin xyz="0 0 0"/>
+            <geometry>
+                <mesh filename="file://$(find robomop_description)/meshes/visual/robomop_brush.stl" scale="0.001 0.001 0.001"/>
+            </geometry>
+            <material name="dark_grey" />
+        </visual>
+        <collision>
+            <origin xyz="0 0 0"/>
+            <geometry>
+                <mesh filename="file://$(find robomop_description)/meshes/visual/robomop_brush.stl" scale="0.001 0.001 0.001"/>
+            </geometry>
+        </collision>
+    </link>
+    <link name="left_brush">
+        <visual>
+            <origin xyz="0 0 0"/>
+            <geometry>
+                <mesh filename="file://$(find robomop_description)/meshes/visual/robomop_brush.stl" scale="0.001 0.001 0.001"/>
+            </geometry>
+            <material name="dark_grey" />
+        </visual>
+        <collision>
+            <origin xyz="0 0 0"/>
+            <geometry>
+                <mesh filename="file://$(find robomop_description)/meshes/visual/robomop_brush.stl" scale="0.001 0.001 0.001"/>
+            </geometry>
+        </collision>
+    </link>
+    <link name="caster_housing">
+        <visual>
+            <origin xyz="0 ${0.047/2} 0" rpy="0 3.14 1.57"/>
+            <geometry>
+                <mesh filename="file://$(find robomop_description)/meshes/visual/robomop_caster.stl" scale="0.001 0.001 0.001"/>
+            </geometry>
+            <material name="grey" />
+        </visual>
+        <collision>
+            <origin xyz="0 ${0.047/2} 0" rpy="0 3.14 1.57"/>
+            <geometry>
+                <mesh filename="file://$(find robomop_description)/meshes/visual/robomop_caster.stl" scale="0.001 0.001 0.001"/>
+            </geometry>
+        </collision>
+    </link>
+    <link name="caster_wheel">
+        <visual>
+            <origin xyz="${(-23.619)/1000} ${16.211/1000} ${(-13.5)/1000}"/>
+            <geometry>
+                <mesh filename="file://$(find robomop_description)/meshes/visual/robomop_caster_wheel.stl" scale="0.001 0.001 0.001"/>
+            </geometry>
+            <material name="grey" />
+        </visual>
+        <collision>
+            <origin xyz="0 0 0"/>
+            <geometry>
+                <mesh filename="file://$(find robomop_description)/meshes/visual/robomop_caster_wheel.stl" scale="0.001 0.001 0.001"/>
+            </geometry>
+        </collision>
+    </link>
     <!-- Lidar Link -->
     <xacro:include filename="$(find ldlidar_node)/urdf/ldlidar_descr.urdf.xml" />
@@ -92,4 +152,26 @@
         <axis xyz="0 1 0"/>
         <origin xyz="${wheel_x_offset} ${-wheel_y_offset - 0.022} ${wheel_z_offset}" rpy="0 0 0" />
+    </joint>
+    <joint name="right_brush_to_chassis" type="continuous">
+        <parent link="chassis_link"/>
+        <child link="right_brush"/>
+        <axis xyz="0 0 1"/>
+        <origin xyz="0.1067 -0.0762 -0.016" rpy="0 0 0" />
+    </joint>
+    <joint name="left_brush_to_chassis" type="continuous">
+        <parent link="chassis_link"/>
+        <child link="left_brush"/>
+        <axis xyz="0 0 1"/>
+        <origin xyz="0.1067 0.0762 -0.016" rpy="0 0 0" />
+    </joint>
+    <joint name="caster_housing_to_chassis" type="fixed">
+        <parent link="chassis_link"/>
+        <child link="caster_housing"/>
+        <origin xyz="${(149.9 - 23.62)/1000} ${0} ${(-14.00)/1000}" rpy="0 0 0" />
+    </joint>
+    <joint name="caster_wheel_to_housing" type="fixed">
+        <parent link="caster_housing"/>
+        <child link="caster_wheel"/>
+        <origin xyz="${16.211/1000} 0 ${(-13)/1000}" rpy="0 0 0" />
     </joint>
     <joint name="lidar_to_chassis" type="fixed">

Commit message: add odometry kinematics and more

File: src/robomop_description/urdf/robomop.urdf.xacro (robot description, xacro)
@@ -31,4 +31,6 @@
         </inertial>
     </link>
+    <link name="chassis_icr_link" /> <!-- center of rotation link for wheels-->
+    <link name="imu_link" />
     <link name="rl_wheel_link">
         <visual>
@@ -141,15 +143,25 @@
         <origin xyz="0 0 ${0.006 + 0.018}"/>
     </joint>
+    <joint name="chassis_to_imu" type="fixed">
+        <parent link="chassis_link"/>
+        <child link="imu_link"/>
+        <origin xyz="-0.02 0 ${wheel_z_offset + 0.025}"/>
+    </joint>
+    <joint name="chassis_to_chassis_icr" type="fixed">
+        <parent link="chassis_link"/>
+        <child link="chassis_icr_link"/>
+        <origin xyz="${wheel_x_offset} 0 0"/>
+    </joint>
     <joint name="rl_wheel_to_chassis" type="continuous">
-        <parent link="chassis_link"/>
+        <parent link="chassis_icr_link"/>
         <child link="rl_wheel_link"/>
         <axis xyz="0 1 0"/>
-        <origin xyz="${wheel_x_offset} ${wheel_y_offset} ${wheel_z_offset}" rpy="0 0 0" />
+        <origin xyz="0 ${wheel_y_offset} ${wheel_z_offset}" rpy="0 0 0" />
     </joint>
     <joint name="rr_wheel_to_chassis" type="continuous">
-        <parent link="chassis_link"/>
+        <parent link="chassis_icr_link"/>
         <child link="rr_wheel_link"/>
         <axis xyz="0 1 0"/>
-        <origin xyz="${wheel_x_offset} ${-wheel_y_offset - 0.022} ${wheel_z_offset}" rpy="0 0 0" />
+        <origin xyz="0 ${-wheel_y_offset - 0.022} ${wheel_z_offset}" rpy="0 0 0" />
     </joint>
     <joint name="right_brush_to_chassis" type="continuous">
